File: hardware/kicad/_autosave-io.kicad_sch (KiCad schematic)
At the start: 12 parts, among them J1 UART connector, SW1 Reset, U10 74HC595, U11 74HC595, U13 74HC165, U14 74HC00, U15 74HC00, U16 MC68B50, U3 6821

Commit message: Update gitnore
Parts:
- removed C1: 10uF, symbol Device:C_Polarized
- removed D1: 1N5819, Diode_THT:D_DO-41_SOD81_P10.16mm_Horizontal, symbol Diode:1N5819
- removed J1: UART connector, symbol Connector_Generic:Conn_01x07
- removed R1: 3.3k, symbol Device:R
- removed SW1: Reset, symbol Switch:SW_Push
- removed U13: 74HC165, symbol 74xx:74HC165
- removed U14, U15: 74HC00, symbol 74xx:74HC00
- removed U16: MC68B50, Package_DIP:DIP-24_W15.24mm_Socket, symbol Interface_UART:MC68B50
- added U?: MC68B50, Package_DIP:DIP-24_W15.24mm_Socket, symbol Interface_UART:MC68B50
- added U?: 74HC165, symbol 74xx:74HC165
Connections:
- net RX_{status} is gone; now on net SRI_{LATCH}: U10.12 (RCLK)
- net +5V: now also U?.12 (VCC), U?.16 (VCC)
- net A0: now also U?.11 (RS)
- net A7: now also U?.8 (CS0)
- net D0: now also U?.11 (D0), U?.22 (D0)
- net D1: now also U?.12 (D1), U?.21 (D1)
- net D2: now also U?.13 (D2), U?.20 (D2)
- net D3: now also U?.14 (D3), U?.19 (D3)
- net D4: now also U?.18 (D4), U?.3 (D4)
- net D5: now also U?.17 (D5), U?.4 (D5)
- net D6: now also U?.16 (D6), U?.5 (D6)
- net D7: now also U?.15 (D7), U?.6 (D7)
- net E: now also U?.14 (E)
- net GND: now also U?.1 (VSS), U?.23 (~{DCD}), U?.24 (~{CTS}), U?.8 (GND)
- net RX: now also U?.2 (Rx_Data); no longer U10.14 (SER)
- net R/~{W}: now also U?.13 (R/~{W})
- net TX: now also U?.6 (Tx_Data)
- net VMA: now also U?.10 (CS1)
- net ~{IRQ}: now also U?.7 (~{IRQ})
- net CS_{RX0} renamed CS_{SRI0}
- net CS_{RX1} renamed CS_{SRI1}
- net RX_{CLK} renamed SRI_{CLK}
- net RX_{latch} renamed SRI_{LATCH}
- new net CLK_{UART0}: U?.3 (Rx_CLK), U?.4 (Tx_CLK)
- new net CS_{SRO}: U?.1 (~{PL})
- new net SRI_{DATA}: U10.14 (SER)
- new net SRO_{CLK}: U?.2 (CP)
- new net SRO_{DATA}: U?.9 (Q7)
- new net ~{CS_{UART0}}: U?.9 (~{CS2})
Other:
- note added: "PiSo interface"
- note added: "SiPo interface"
- note added: "UART"
- moved on the sheet: U10, U11, U3
