File: hardware/kicad/connectors.kicad_sch (KiCad schematic)
At the start: 1 part

Commit message: Start PCB design
Parts:
- J?: footprint (none) -> Connector_PinHeader_2.54mm:PinHeader_1x04_P2.54mm_Vertical
Changed lines of the file:
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@@
       (effects (font (size 1.27 1.27)) (justify left))
     )
-    (property "Footprint" "" (at 40.64 43.18 0)
+    (property "Footprint" "Connector_PinHeader_2.54mm:PinHeader_1x04_P2.54mm_Vertical" (at 40.64 43.18 0)
       (effects (font (size 1.27 1.27)) hide)
     )
@@
         )
         (path "/e63e39d7-6ac0-4ffd-8aa3-1841a4541b55/333dc95e-1212-4562-83c9-7eee6e0243bf"
-          (reference "J?") (unit 1)
+          (reference "J1") (unit 1)
         )
       )
@@
   (symbol (lib_id "power:+5V") (at 35.56 40.64 0) (unit 1)
     (in_bom yes) (on_board yes) (dnp no) (fields_autoplaced)
-    (property "Reference" "#PWR041" (at 35.56 44.45 0)
+    (property "Reference" "#PWR01" (at 35.56 44.45 0)
       (effects (font (size 1.27 1.27)) hide)
     )
@@
       (project "6802 v1"
         (path "/e63e39d7-6ac0-4ffd-8aa3-1841a4541b55/333dc95e-1212-4562-83c9-7eee6e0243bf"
-          (reference "#PWR041") (unit 1)
+          (reference "#PWR01") (unit 1)
         )
       )
@@
         )
         (path "/e63e39d7-6ac0-4ffd-8aa3-1841a4541b55/333dc95e-1212-4562-83c9-7eee6e0243bf"
-          (reference "#PWR037") (unit 1)
+          (reference "#PWR02") (unit 1)
         )
       )
