File: hardware/kicad/cpu.kicad_sch (KiCad schematic)
At the start: 7 parts, among them U2 MC6802, Y1 4MHz Crystal

Commit message: Update gitnore
Parts:
- added U1, U5: 74LS245, symbol 74xx:74LS245
- added U14: 74LS138, symbol 74xx:74LS138
- added U9: 74LS138, Package_DIP:DIP-16_W7.62mm_Socket, symbol 74xx:74LS138
Connections:
- net +5V: now also U1.20 (VCC), U14.16 (VCC), U5.20 (VCC), U9.16 (VCC), U9.6 (E3)
- net A0: now also U1.18 (B0)
- net A1: now also U1.17 (B1)
- net A10: now also U5.16 (B2)
- net A11: now also U5.15 (B3), U9.1 (A0)
- net A12: now also U5.14 (B4), U9.2 (A1)
- net A13: now also U5.13 (B5), U9.3 (A2)
- net A14: now also U5.12 (B6), U9.4 (E1)
- net A15: now also U5.11 (B7), U9.5 (E2)
- net A2: now also U1.16 (B2)
- net A3: now also U1.15 (B3), U14.1 (A0)
- net A4: now also U1.14 (B4), U14.2 (A1)
- net A5: now also U1.13 (B5), U14.3 (A2)
- net A6: now also U1.12 (B6)
- net A7: now also U1.11 (B7), U14.6 (E3)
- net A8: now also U14.5 (E2), U5.18 (B0)
- net A9: now also U5.17 (B1)
- net GND: now also U1.1 (A->B), U1.10 (GND), U14.8 (GND), U5.1 (A->B), U5.10 (GND), U9.8 (GND)
- new net A_{b}0: U1.2 (A0)
- new net A_{b}1: U1.3 (A1)
- new net A_{b}10: U5.4 (A2)
- new net A_{b}11: U5.5 (A3)
- new net A_{b}12: U5.6 (A4)
- new net A_{b}13: U5.7 (A5)
- new net A_{b}14: U5.8 (A6)
- new net A_{b}15: U5.9 (A7)
- new net A_{b}2: U1.4 (A2)
- new net A_{b}3: U1.5 (A3)
- new net A_{b}4: U1.6 (A4)
- new net A_{b}5: U1.7 (A5)
- new net A_{b}6: U1.8 (A6)
- new net A_{b}7: U1.9 (A7)
- new net A_{b}8: U5.2 (A0)
- new net A_{b}9: U5.3 (A1)
- new net CS_{RX0}: U14.14 (O1)
- new net CS_{RX1}: U14.13 (O2)
- new net CS_{TX0}: U14.12 (O3)
- new net CS_{TX1}: U14.11 (O4)
- new net DMA: U1.19 (CE), U5.19 (CE)
- new net ~{CS^{13}_{0}}: U9.14 (O1)
- new net ~{CS^{13}_{1}}: U9.13 (O2)
- new net ~{CS^{13}_{2}}: U9.12 (O3)
- new net ~{CS^{13}_{3}}: U9.11 (O4)
- new net ~{CS^{13}_{4}}: U9.10 (O5)
- new net ~{CS^{13}_{5}}: U9.9 (O6)
- new net ~{CS^{13}_{6}}: U9.7 (O7)
- new net ~{CS^{13}_{H}}: U14.4 (E1), U9.15 (O0)
- new net ~{CS_{PIA}}: U14.15 (O0)
Other:
- note added: "Address decoders"
- note added: "Address line buffers (tri-state)"
- note added: "CPU"

Commit message: Start PCB design
Parts:
- R2, R3, R4: footprint (none) -> Resistor_THT:R_Axial_DIN0207_L6.3mm_D2.5mm_P10.16mm_Horizontal
- U1, U5: footprint (none) -> Package_DIP:DIP-20_W7.62mm_Socket
- U14: footprint (none) -> Package_DIP:DIP-16_W7.62mm_Socket
Changed lines of the file:
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@@
       (effects (font (size 1.27 1.27)) (justify left))
     )
-    (property "Footprint" "" (at 97.79 156.21 0)
+    (property "Footprint" "Package_DIP:DIP-20_W7.62mm_Socket" (at 97.79 156.21 0)
       (effects (font (size 1.27 1.27)) hide)
     )
@@
         )
         (path "/e63e39d7-6ac0-4ffd-8aa3-1841a4541b55/366e0d9a-56e6-4430-93d3-3a271557a8cc"
-          (reference "U5") (unit 1)
+          (reference "U12") (unit 1)
         )
       )
@@
         )
         (path "/e63e39d7-6ac0-4ffd-8aa3-1841a4541b55/366e0d9a-56e6-4430-93d3-3a271557a8cc"
-          (reference "#PWR025") (unit 1)
+          (reference "#PWR036") (unit 1)
         )
       )
@@
         )
         (path "/e63e39d7-6ac0-4ffd-8aa3-1841a4541b55/366e0d9a-56e6-4430-93d3-3a271557a8cc"
-          (reference "#PWR013") (unit 1)
+          (reference "#PWR028") (unit 1)
         )
       )
@@
         )
         (path "/e63e39d7-6ac0-4ffd-8aa3-1841a4541b55/366e0d9a-56e6-4430-93d3-3a271557a8cc"
-          (reference "#PWR026") (unit 1)
+          (reference "#PWR027") (unit 1)
         )
       )
@@
         )
         (path "/e63e39d7-6ac0-4ffd-8aa3-1841a4541b55/366e0d9a-56e6-4430-93d3-3a271557a8cc"
-          (reference "C3") (unit 1)
+          (reference "C2") (unit 1)
         )
       )
@@
       (effects (font (size 1.27 1.27)))
     )
-    (property "Footprint" "" (at 35.79 66.318 90)
+    (property "Footprint" "Resistor_THT:R_Axial_DIN0207_L6.3mm_D2.5mm_P10.16mm_Horizontal" (at 35.79 66.318 90)
       (effects (font (size 1.27 1.27)) hide)
     )
@@
         )
         (path "/e63e39d7-6ac0-4ffd-8aa3-1841a4541b55/366e0d9a-56e6-4430-93d3-3a271557a8cc"
-          (reference "R3") (unit 1)
+          (reference "R2") (unit 1)
         )
       )
@@
         )
         (path "/e63e39d7-6ac0-4ffd-8aa3-1841a4541b55/366e0d9a-56e6-4430-93d3-3a271557a8cc"
-          (reference "#PWR012") (unit 1)
+          (reference "#PWR025") (unit 1)
         )
       )
@@
         )
         (path "/e63e39d7-6ac0-4ffd-8aa3-1841a4541b55/366e0d9a-56e6-4430-93d3-3a271557a8cc"
-          (reference "#PWR028") (unit 1)
+          (reference "#PWR038") (unit 1)
         )
       )
@@
         )
         (path "/e63e39d7-6ac0-4ffd-8aa3-1841a4541b55/366e0d9a-56e6-4430-93d3-3a271557a8cc"
-          (reference "#PWR01") (unit 1)
+          (reference "#PWR021") (unit 1)
         )
       )
@@
         )
         (path "/e63e39d7-6ac0-4ffd-8aa3-1841a4541b55/366e0d9a-56e6-4430-93d3-3a271557a8cc"
-          (reference "U2") (unit 1)
+          (reference "U10") (unit 1)
         )
       )
@@
       (effects (font (size 1.27 1.27)) (justify left))
     )
-    (property "Footprint" "" (at 119.75 39.91 0)
+    (property "Footprint" "Package_DIP:DIP-16_W7.62mm_Socket" (at 119.75 39.91 0)
       (effects (font (size 1.27 1.27)) hide)
     )
@@
         )
         (path "/e63e39d7-6ac0-4ffd-8aa3-1841a4541b55/366e0d9a-56e6-4430-93d3-3a271557a8cc"
-          (reference "U1") (unit 1)
+          (reference "U9") (unit 1)
         )
       )
@@
         )
         (path "/e63e39d7-6ac0-4ffd-8aa3-1841a4541b55/366e0d9a-56e6-4430-93d3-3a271557a8cc"
-          (reference "#PWR031") (unit 1)
+          (reference "#PWR032") (unit 1)
         )
       )
@@
         )
         (path "/e63e39d7-6ac0-4ffd-8aa3-1841a4541b55/366e0d9a-56e6-4430-93d3-3a271557a8cc"
-          (reference "C2") (unit 1)
+          (reference "C1") (unit 1)
         )
       )
@@
         )
         (path "/e63e39d7-6ac0-4ffd-8aa3-1841a4541b55/366e0d9a-56e6-4430-93d3-3a271557a8cc"
-          (reference "#PWR09") (unit 1)
+          (reference "#PWR034") (unit 1)
         )
       )
@@
         )
         (path "/e63e39d7-6ac0-4ffd-8aa3-1841a4541b55/366e0d9a-56e6-4430-93d3-3a271557a8cc"
-          (reference "U12") (unit 1)
+          (reference "U11") (unit 1)
         )
       )
@@
         )
         (path "/e63e39d7-6ac0-4ffd-8aa3-1841a4541b55/366e0d9a-56e6-4430-93d3-3a271557a8cc"
-          (reference "#PWR02") (unit 1)
+          (reference "#PWR022") (unit 1)
         )
       )
@@
         )
         (path "/e63e39d7-6ac0-4ffd-8aa3-1841a4541b55/366e0d9a-56e6-4430-93d3-3a271557a8cc"
-          (reference "#PWR014") (unit 1)
+          (reference "#PWR029") (unit 1)
         )
       )
@@
         )
         (path "/e63e39d7-6ac0-4ffd-8aa3-1841a4541b55/366e0d9a-56e6-4430-93d3-3a271557a8cc"
-          (reference "#PWR03") (unit 1)
+          (reference "#PWR033") (unit 1)
         )
       )
@@
       (effects (font (size 1.27 1.27)))
     )
-    (property "Footprint" "" (at 35.79 63.778 90)
+    (property "Footprint" "Resistor_THT:R_Axial_DIN0207_L6.3mm_D2.5mm_P10.16mm_Horizontal" (at 35.79 63.778 90)
       (effects (font (size 1.27 1.27)) hide)
     )
@@
         )
         (path "/e63e39d7-6ac0-4ffd-8aa3-1841a4541b55/366e0d9a-56e6-4430-93d3-3a271557a8cc"
-          (reference "R2") (unit 1)
+          (reference "R1") (unit 1)
         )
       )
@@
         )
         (path "/e63e39d7-6ac0-4ffd-8aa3-1841a4541b55/366e0d9a-56e6-4430-93d3-3a271557a8cc"
-          (reference "#PWR011") (unit 1)
+          (reference "#PWR023") (unit 1)
         )
       )
@@
         )
         (path "/e63e39d7-6ac0-4ffd-8aa3-1841a4541b55/366e0d9a-56e6-4430-93d3-3a271557a8cc"
-          (reference "#PWR017") (unit 1)
+          (reference "#PWR035") (unit 1)
         )
       )
@@
         )
         (path "/e63e39d7-6ac0-4ffd-8aa3-1841a4541b55/366e0d9a-56e6-4430-93d3-3a271557a8cc"
-          (reference "#PWR08") (unit 1)
+          (reference "#PWR024") (unit 1)
         )
       )
@@
       (effects (font (size 1.27 1.27)))
     )
-    (property "Footprint" "" (at 35.79 68.858 90)
+    (property "Footprint" "Resistor_THT:R_Axial_DIN0207_L6.3mm_D2.5mm_P10.16mm_Horizontal" (at 35.79 68.858 90)
       (effects (font (size 1.27 1.27)) hide)
     )
@@
         )
         (path "/e63e39d7-6ac0-4ffd-8aa3-1841a4541b55/366e0d9a-56e6-4430-93d3-3a271557a8cc"
-          (reference "R4") (unit 1)
+          (reference "R3") (unit 1)
         )
       )
@@
         )
         (path "/e63e39d7-6ac0-4ffd-8aa3-1841a4541b55/366e0d9a-56e6-4430-93d3-3a271557a8cc"
-          (reference "#PWR010") (unit 1)
+          (reference "#PWR026") (unit 1)
         )
       )
@@
       (effects (font (size 1.27 1.27)) (justify left))
     )
-    (property "Footprint" "" (at 50.8 157.48 0)
+    (property "Footprint" "Package_DIP:DIP-20_W7.62mm_Socket" (at 50.8 157.48 0)
       (effects (font (size 1.27 1.27)) hide)
     )
@@
         )
         (path "/e63e39d7-6ac0-4ffd-8aa3-1841a4541b55/366e0d9a-56e6-4430-93d3-3a271557a8cc"
-          (reference "U9") (unit 1)
+          (reference "U13") (unit 1)
         )
       )
@@
         )
         (path "/e63e39d7-6ac0-4ffd-8aa3-1841a4541b55/366e0d9a-56e6-4430-93d3-3a271557a8cc"
-          (reference "#PWR027") (unit 1)
+          (reference "#PWR037") (unit 1)
         )
       )
@@
         )
         (path "/e63e39d7-6ac0-4ffd-8aa3-1841a4541b55/366e0d9a-56e6-4430-93d3-3a271557a8cc"
-          (reference "#PWR016") (unit 1)
-        )
-      )
+          (reference "#PWR031") (unit 1)
+        )
+      )
