File: hardware/kicad/gluelogic.kicad_sch (KiCad schematic)
At the start: 6 parts, among them SW1 Reset, U4 74LS04

Commit message: Start PCB design
Parts:
- C1: footprint (none) -> Capacitor_THT:CP_Radial_D5.0mm_P2.00mm
- R1: footprint (none) -> Resistor_THT:R_Axial_DIN0207_L6.3mm_D2.5mm_P10.16mm_Horizontal
- SW1: footprint (none) -> Button_Switch_THT:SW_PUSH_6mm
- U15: renamed from U?; footprint Package_DIP:DIP-12_W7.62mm_Socket -> Package_DIP:DIP-14_W7.62mm_Socket
- U4: footprint (none) -> Package_DIP:DIP-14_W7.62mm_Socket
Changed lines of the file:
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@@
   (symbol (lib_id "74xx:74LS90") (at 33.02 175.26 0) (unit 1)
     (in_bom yes) (on_board yes) (dnp no) (fields_autoplaced)
-    (property "Reference" "U?" (at 34.9759 161.29 0)
+    (property "Reference" "U15" (at 34.9759 161.29 0)
       (effects (font (size 1.27 1.27)) (justify left) hide)
     )
@@
       (effects (font (size 1.27 1.27)) (justify left))
     )
-    (property "Footprint" "Package_DIP:DIP-12_W7.62mm_Socket" (at 33.02 175.26 0)
+    (property "Footprint" "Package_DIP:DIP-14_W7.62mm_Socket" (at 33.02 175.26 0)
       (effects (font (size 1.27 1.27)) hide)
     )
@@
       (project "6802 v1"
         (path "/e63e39d7-6ac0-4ffd-8aa3-1841a4541b55/bed2405d-2e60-4918-bd56-516da766b029"
-          (reference "U?") (unit 1)
+          (reference "U15") (unit 1)
         )
       )
@@
         )
         (path "/e63e39d7-6ac0-4ffd-8aa3-1841a4541b55/bed2405d-2e60-4918-bd56-516da766b029"
-          (reference "D?") (unit 1)
+          (reference "D1") (unit 1)
         )
       )
@@
         )
         (path "/e63e39d7-6ac0-4ffd-8aa3-1841a4541b55/bed2405d-2e60-4918-bd56-516da766b029"
-          (reference "#PWR07") (unit 1)
+          (reference "#PWR041") (unit 1)
         )
       )
@@
   (symbol (lib_id "power:+5V") (at 33.02 160.02 0) (unit 1)
     (in_bom yes) (on_board yes) (dnp no) (fields_autoplaced)
-    (property "Reference" "#PWR044" (at 33.02 163.83 0)
+    (property "Reference" "#PWR042" (at 33.02 163.83 0)
       (effects (font (size 1.27 1.27)) hide)
     )
@@
       (project "6802 v1"
         (path "/e63e39d7-6ac0-4ffd-8aa3-1841a4541b55/bed2405d-2e60-4918-bd56-516da766b029"
-          (reference "#PWR044") (unit 1)
+          (reference "#PWR042") (unit 1)
         )
       )
@@
       (effects (font (size 1.27 1.27)) (justify right))
     )
-    (property "Footprint" "" (at 37.338 119.38 90)
+    (property "Footprint" "Resistor_THT:R_Axial_DIN0207_L6.3mm_D2.5mm_P10.16mm_Horizontal" (at 37.338 119.38 90)
       (effects (font (size 1.27 1.27)) hide)
     )
@@
         )
         (path "/e63e39d7-6ac0-4ffd-8aa3-1841a4541b55/bed2405d-2e60-4918-bd56-516da766b029"
-          (reference "R?") (unit 1)
+          (reference "R4") (unit 1)
         )
       )
@@
         )
         (path "/e63e39d7-6ac0-4ffd-8aa3-1841a4541b55/bed2405d-2e60-4918-bd56-516da766b029"
-          (reference "#PWR06") (unit 1)
+          (reference "#PWR040") (unit 1)
         )
       )
@@
       (effects (font (size 1.27 1.27)) (justify right))
     )
-    (property "Footprint" "" (at 20.32 129.54 0)
+    (property "Footprint" "Button_Switch_THT:SW_PUSH_6mm" (at 20.32 129.54 0)
       (effects (font (size 1.27 1.27)) hide)
     )
@@
         )
         (path "/e63e39d7-6ac0-4ffd-8aa3-1841a4541b55/bed2405d-2e60-4918-bd56-516da766b029"
-          (reference "SW?") (unit 1)
+          (reference "SW1") (unit 1)
         )
       )
@@
         )
         (path "/e63e39d7-6ac0-4ffd-8aa3-1841a4541b55/bed2405d-2e60-4918-bd56-516da766b029"
-          (reference "#PWR05") (unit 1)
+          (reference "#PWR039") (unit 1)
         )
       )
@@
   (symbol (lib_id "power:GND") (at 17.78 185.42 0) (unit 1)
     (in_bom yes) (on_board yes) (dnp no) (fields_autoplaced)
-    (property "Reference" "#PWR042" (at 17.78 191.77 0)
+    (property "Reference" "#PWR043" (at 17.78 191.77 0)
       (effects (font (size 1.27 1.27)) hide)
     )
@@
       (project "6802 v1"
         (path "/e63e39d7-6ac0-4ffd-8aa3-1841a4541b55/bed2405d-2e60-4918-bd56-516da766b029"
-          (reference "#PWR042") (unit 1)
+          (reference "#PWR043") (unit 1)
         )
       )
@@
         )
         (path "/e63e39d7-6ac0-4ffd-8aa3-1841a4541b55/bed2405d-2e60-4918-bd56-516da766b029"
-          (reference "U4") (unit 2)
+          (reference "U14") (unit 2)
         )
       )
@@
       (effects (font (size 1.27 1.27)))
     )
-    (property "Footprint" "" (at 36.5252 133.35 0)
+    (property "Footprint" "Capacitor_THT:CP_Radial_D5.0mm_P2.00mm" (at 36.5252 133.35 0)
       (effects (font (size 1.27 1.27)) hide)
     )
@@
         )
         (path "/e63e39d7-6ac0-4ffd-8aa3-1841a4541b55/bed2405d-2e60-4918-bd56-516da766b029"
-          (reference "C?") (unit 1)
+          (reference "C3") (unit 1)
         )
       )
@@
   (symbol (lib_id "power:GND") (at 33.02 193.04 0) (unit 1)
     (in_bom yes) (on_board yes) (dnp no) (fields_autoplaced)
-    (property "Reference" "#PWR043" (at 33.02 199.39 0)
+    (property "Reference" "#PWR044" (at 33.02 199.39 0)
       (effects (font (size 1.27 1.27)) hide)
     )
@@
       (project "6802 v1"
         (path "/e63e39d7-6ac0-4ffd-8aa3-1841a4541b55/bed2405d-2e60-4918-bd56-516da766b029"
-          (reference "#PWR043") (unit 1)
+          (reference "#PWR044") (unit 1)
         )
       )
@@
       (effects (font (size 1.27 1.27)) hide)
     )
-    (property "Footprint" "" (at 43.18 43.18 0)
+    (property "Footprint" "Package_DIP:DIP-14_W7.62mm_Socket" (at 43.18 43.18 0)
       (effects (font (size 1.27 1.27)) hide)
     )
@@
         )
         (path "/e63e39d7-6ac0-4ffd-8aa3-1841a4541b55/bed2405d-2e60-4918-bd56-516da766b029"
-          (reference "U4") (unit 1)
-        )
-      )
+          (reference "U14") (unit 1)
+        )
+      )
