File: hardware/kicad/io.kicad_sch (KiCad schematic)
At the start: 11 parts, among them J1 UART connector, SW1 Reset, U10 74HC595, U11 74HC595, U13 74HC165, U14 74HC00, U15 74HC00, U3 6821

Commit message: Update gitnore
Parts:
- removed C1: 10uF, symbol Device:C_Polarized
- removed D1: 1N5819, Diode_THT:D_DO-41_SOD81_P10.16mm_Horizontal, symbol Diode:1N5819
- removed J1: UART connector, symbol Connector_Generic:Conn_01x07
- removed R1: 3.3k, symbol Device:R
- removed SW1: Reset, symbol Switch:SW_Push
- removed U13: 74HC165, symbol 74xx:74HC165
- removed U14, U15: 74HC00, symbol 74xx:74HC00
- added U?: MC68B50, Package_DIP:DIP-24_W15.24mm_Socket, symbol Interface_UART:MC68B50
- added U?: 74HC165, symbol 74xx:74HC165
Connections:
- net RX_{status} is gone; now on net SRI_{LATCH}: U10.12 (RCLK)
- net +5V: now also U?.12 (VCC), U?.16 (VCC)
- net A0: now also U?.11 (RS)
- net A7: now also U?.8 (CS0)
- net D0: now also U?.11 (D0), U?.22 (D0)
- net D1: now also U?.12 (D1), U?.21 (D1)
- net D2: now also U?.13 (D2), U?.20 (D2)
- net D3: now also U?.14 (D3), U?.19 (D3)
- net D4: now also U?.18 (D4), U?.3 (D4)
- net D5: now also U?.17 (D5), U?.4 (D5)
- net D6: now also U?.16 (D6), U?.5 (D6)
- net D7: now also U?.15 (D7), U?.6 (D7)
- net E: now also U?.14 (E)
- net GND: now also U?.1 (VSS), U?.23 (~{DCD}), U?.24 (~{CTS}), U?.8 (GND)
- net RX: now also U?.2 (Rx_Data); no longer U10.14 (SER)
- net R/~{W}: now also U?.13 (R/~{W})
- net TX: now also U?.6 (Tx_Data)
- net VMA: now also U?.10 (CS1)
- net ~{IRQ}: now also U?.7 (~{IRQ})
- net CS_{RX0} renamed CS_{SRI0}
- net CS_{RX1} renamed CS_{SRI1}
- net RX_{CLK} renamed SRI_{CLK}
- net RX_{latch} renamed SRI_{LATCH}
- new net CLK_{UART0}: U?.3 (Rx_CLK), U?.4 (Tx_CLK)
- new net CS_{SRO}: U?.1 (~{PL})
- new net SRI_{DATA}: U10.14 (SER)
- new net SRO_{CLK}: U?.2 (CP)
- new net SRO_{DATA}: U?.9 (Q7)
- new net ~{CS_{UART0}}: U?.9 (~{CS2})
Other:
- moved on the sheet: U10, U11, U3

Commit message: Cont
Other:
- note added: "PiSo interface"
- note added: "SiPo interface"
- note added: "UART"
Changed lines of the file:
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@@
     (stroke (width 0) (type default))
+  )
+  (text "SiPo interface" (at 81.28 91.44 0)
+    (effects (font (size 1.5 1.5) bold) (justify left bottom))
+  )
+  (text "PiSo interface" (at 73.66 15.24 0)
+    (effects (font (size 1.5 1.5) bold) (justify left bottom))
+  )
+  (text "UART" (at 30.48 17.78 0)
+    (effects (font (size 1.5 1.5) bold) (justify left bottom))
   )
   (global_label "D2" (shape bidirectional) (at 25.4 33.02 180) (fields_autoplaced)

Commit message: Start PCB design
Parts:
- U4: renamed from U?; footprint (none) -> Package_DIP:DIP-16_W7.62mm_Socket
- gave numbers to parts that had none: 1
- renumbered U10 to U7, U11 to U8
Changed lines of the file:
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@@
         )
         (path "/e63e39d7-6ac0-4ffd-8aa3-1841a4541b55/aacad567-86ad-4193-8aa8-08565ab103a5"
-          (reference "#PWR015") (unit 1)
+          (reference "#PWR016") (unit 1)
         )
       )
@@
   (symbol (lib_id "power:+5V") (at 38.1 22.86 0) (unit 1)
     (in_bom yes) (on_board yes) (dnp no) (fields_autoplaced)
-    (property "Reference" "#PWR038" (at 38.1 26.67 0)
+    (property "Reference" "#PWR011" (at 38.1 26.67 0)
       (effects (font (size 1.27 1.27)) hide)
     )
@@
       (project "6802 v1"
         (path "/e63e39d7-6ac0-4ffd-8aa3-1841a4541b55/aacad567-86ad-4193-8aa8-08565ab103a5"
-          (reference "#PWR038") (unit 1)
+          (reference "#PWR011") (unit 1)
         )
       )
@@
         )
         (path "/e63e39d7-6ac0-4ffd-8aa3-1841a4541b55/aacad567-86ad-4193-8aa8-08565ab103a5"
-          (reference "#PWR04") (unit 1)
+          (reference "#PWR012") (unit 1)
         )
       )
@@
   (symbol (lib_id "Interface_UART:MC68B50") (at 38.1 55.88 0) (unit 1)
     (in_bom yes) (on_board yes) (dnp no) (fields_autoplaced)
-    (property "Reference" "U?" (at 40.0559 21.91 0)
+    (property "Reference" "U5" (at 40.0559 21.91 0)
       (effects (font (size 1.27 1.27)) (justify left) hide)
     )
@@
       (project "6802 v1"
         (path "/e63e39d7-6ac0-4ffd-8aa3-1841a4541b55/aacad567-86ad-4193-8aa8-08565ab103a5"
-          (reference "U?") (unit 1)
+          (reference "U5") (unit 1)
         )
       )
@@
   (symbol (lib_name "GND_1") (lib_id "power:GND") (at 88.16 177.93 0) (unit 1)
     (in_bom yes) (on_board yes) (dnp no) (fields_autoplaced)
-    (property "Reference" "#PWR034" (at 88.16 184.28 0)
+    (property "Reference" "#PWR020" (at 88.16 184.28 0)
       (effects (font (size 1.27 1.27)) hide)
     )
@@
       (project "6802 v1"
         (path "/e63e39d7-6ac0-4ffd-8aa3-1841a4541b55/aacad567-86ad-4193-8aa8-08565ab103a5"
-          (reference "#PWR034") (unit 1)
+          (reference "#PWR020") (unit 1)
         )
       )
@@
         )
         (path "/e63e39d7-6ac0-4ffd-8aa3-1841a4541b55/aacad567-86ad-4193-8aa8-08565ab103a5"
-          (reference "U3") (unit 1)
+          (reference "U6") (unit 1)
         )
       )
@@
   (symbol (lib_name "GND_2") (lib_id "power:GND") (at 86.43 68.7 0) (unit 1)
     (in_bom yes) (on_board yes) (dnp no) (fields_autoplaced)
-    (property "Reference" "#PWR036" (at 86.43 75.05 0)
+    (property "Reference" "#PWR013" (at 86.43 75.05 0)
       (effects (font (size 1.27 1.27)) hide)
     )
@@
       (project "6802 v1"
         (path "/e63e39d7-6ac0-4ffd-8aa3-1841a4541b55/aacad567-86ad-4193-8aa8-08565ab103a5"
-          (reference "#PWR036") (unit 1)
+          (reference "#PWR013") (unit 1)
         )
       )
@@
   (symbol (lib_id "74xx:74HC595") (at 88.16 160.15 0) (unit 1)
     (in_bom yes) (on_board yes) (dnp no) (fields_autoplaced)
-    (property "Reference" "U11" (at 90.1159 143.64 0)
+    (property "Reference" "U8" (at 90.1159 143.64 0)
       (effects (font (size 1.27 1.27)) (justify left))
     )
@@
       (project "6802 v1"
         (path "/e63e39d7-6ac0-4ffd-8aa3-1841a4541b55/aacad567-86ad-4193-8aa8-08565ab103a5"
-          (reference "U11") (unit 1)
+          (reference "U8") (unit 1)
         )
       )
@@
   (symbol (lib_name "+5V_1") (lib_id "power:+5V") (at 88.16 144.91 0) (unit 1)
     (in_bom yes) (on_board yes) (dnp no) (fields_autoplaced)
-    (property "Reference" "#PWR032" (at 88.16 148.72 0)
+    (property "Reference" "#PWR019" (at 88.16 148.72 0)
       (effects (font (size 1.27 1.27)) hide)
     )
@@
       (project "6802 v1"
         (path "/e63e39d7-6ac0-4ffd-8aa3-1841a4541b55/aacad567-86ad-4193-8aa8-08565ab103a5"
-          (reference "#PWR032") (unit 1)
+          (reference "#PWR019") (unit 1)
         )
       )
@@
   (symbol (lib_name "GND_1") (lib_id "power:GND") (at 88.16 130.94 0) (unit 1)
     (in_bom yes) (on_board yes) (dnp no) (fields_autoplaced)
-    (property "Reference" "#PWR035" (at 88.16 137.29 0)
+    (property "Reference" "#PWR018" (at 88.16 137.29 0)
       (effects (font (size 1.27 1.27)) hide)
     )
@@
       (project "6802 v1"
         (path "/e63e39d7-6ac0-4ffd-8aa3-1841a4541b55/aacad567-86ad-4193-8aa8-08565ab103a5"
-          (reference "#PWR035") (unit 1)
+          (reference "#PWR018") (unit 1)
         )
       )
@@
   (symbol (lib_name "+5V_2") (lib_id "power:+5V") (at 86.43 20.44 0) (unit 1)
     (in_bom yes) (on_board yes) (dnp no) (fields_autoplaced)
-    (property "Reference" "#PWR033" (at 86.43 24.25 0)
+    (property "Reference" "#PWR010" (at 86.43 24.25 0)
       (effects (font (size 1.27 1.27)) hide)
     )
@@
       (project "6802 v1"
         (path "/e63e39d7-6ac0-4ffd-8aa3-1841a4541b55/aacad567-86ad-4193-8aa8-08565ab103a5"
-          (reference "#PWR033") (unit 1)
+          (reference "#PWR010") (unit 1)
         )
       )
@@
   (symbol (lib_name "+5V_1") (lib_id "power:+5V") (at 88.16 97.92 0) (unit 1)
     (in_bom yes) (on_board yes) (dnp no) (fields_autoplaced)
-    (property "Reference" "#PWR029" (at 88.16 101.73 0)
+    (property "Reference" "#PWR017" (at 88.16 101.73 0)
       (effects (font (size 1.27 1.27)) hide)
     )
@@
       (project "6802 v1"
         (path "/e63e39d7-6ac0-4ffd-8aa3-1841a4541b55/aacad567-86ad-4193-8aa8-08565ab103a5"
-          (reference "#PWR029") (unit 1)
+          (reference "#PWR017") (unit 1)
         )
       )
@@
   (symbol (lib_id "power:GND") (at 25.4 81.28 0) (unit 1)
     (in_bom yes) (on_board yes) (dnp no) (fields_autoplaced)
-    (property "Reference" "#PWR040" (at 25.4 87.63 0)
+    (property "Reference" "#PWR014" (at 25.4 87.63 0)
       (effects (font (size 1.27 1.27)) hide)
     )
@@
       (project "6802 v1"
         (path "/e63e39d7-6ac0-4ffd-8aa3-1841a4541b55/aacad567-86ad-4193-8aa8-08565ab103a5"
-          (reference "#PWR040") (unit 1)
+          (reference "#PWR014") (unit 1)
         )
       )
@@
   (symbol (lib_id "74xx:74HC595") (at 88.16 113.16 0) (unit 1)
     (in_bom yes) (on_board yes) (dnp no) (fields_autoplaced)
-    (property "Reference" "U10" (at 90.1159 96.65 0)
+    (property "Reference" "U7" (at 90.1159 96.65 0)
       (effects (font (size 1.27 1.27)) (justify left))
     )
@@
       (project "6802 v1"
         (path "/e63e39d7-6ac0-4ffd-8aa3-1841a4541b55/aacad567-86ad-4193-8aa8-08565ab103a5"
-          (reference "U10") (unit 1)
+          (reference "U7") (unit 1)
         )
       )
@@
   (symbol (lib_id "power:GND") (at 38.1 86.36 0) (unit 1)
     (in_bom yes) (on_board yes) (dnp no) (fields_autoplaced)
-    (property "Reference" "#PWR039" (at 38.1 92.71 0)
+    (property "Reference" "#PWR015" (at 38.1 92.71 0)
       (effects (font (size 1.27 1.27)) hide)
     )
@@
       (project "6802 v1"
         (path "/e63e39d7-6ac0-4ffd-8aa3-1841a4541b55/aacad567-86ad-4193-8aa8-08565ab103a5"
-          (reference "#PWR039") (unit 1)
+          (reference "#PWR015") (unit 1)
         )
       )
@@
   (symbol (lib_id "74xx:74HC165") (at 86.36 43.18 0) (mirror y) (unit 1)
     (in_bom yes) (on_board yes) (dnp no)
-    (property "Reference" "U?" (at 84.4041 21.59 0)
+    (property "Reference" "U4" (at 84.4041 21.59 0)
       (effects (font (size 1.27 1.27)) (justify left))
     )
@@
       (effects (font (size 1.27 1.27)) (justify left))
     )
-    (property "Footprint" "" (at 86.36 43.18 0)
+    (property "Footprint" "Package_DIP:DIP-16_W7.62mm_Socket" (at 86.36 43.18 0)
       (effects (font (size 1.27 1.27)) hide)
     )
@@
       (project "6802 v1"
         (path "/e63e39d7-6ac0-4ffd-8aa3-1841a4541b55/aacad567-86ad-4193-8aa8-08565ab103a5"
-          (reference "U?") (unit 1)
-        )
-      )
+          (reference "U4") (unit 1)
+        )
+      )
