File: hardware/kicad/memory.kicad_sch (KiCad schematic)
At the start: 8 parts, among them U1 74LS245, U14 74LS138, U4 74LS04, U5 74LS245, U6 UM6116, U7 27C512, U8 UM6116, U9 74LS138

Commit message: Update gitnore
Parts:
- removed U1, U5: 74LS245, symbol 74xx:74LS245
- removed U14: 74LS138, symbol 74xx:74LS138
- removed U4: 74LS04, symbol 74xx:74LS04
- removed U9: 74LS138, Package_DIP:DIP-16_W7.62mm_Socket, symbol 74xx:74LS138

Commit message: Start PCB design
Parts:
- U6, U8: footprint (none) -> Package_DIP:DIP-24_W15.24mm_Socket
Changed lines of the file:
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@@
         )
         (path "/e63e39d7-6ac0-4ffd-8aa3-1841a4541b55/bfe21baf-1342-48ad-994b-20326b13bad2"
-          (reference "#PWR021") (unit 1)
+          (reference "#PWR06") (unit 1)
         )
       )
@@
         )
         (path "/e63e39d7-6ac0-4ffd-8aa3-1841a4541b55/bfe21baf-1342-48ad-994b-20326b13bad2"
-          (reference "#PWR022") (unit 1)
+          (reference "#PWR07") (unit 1)
         )
       )
@@
         )
         (path "/e63e39d7-6ac0-4ffd-8aa3-1841a4541b55/bfe21baf-1342-48ad-994b-20326b13bad2"
-          (reference "#PWR023") (unit 1)
+          (reference "#PWR08") (unit 1)
         )
       )
@@
         )
         (path "/e63e39d7-6ac0-4ffd-8aa3-1841a4541b55/bfe21baf-1342-48ad-994b-20326b13bad2"
-          (reference "#PWR018") (unit 1)
+          (reference "#PWR03") (unit 1)
         )
       )
@@
         )
         (path "/e63e39d7-6ac0-4ffd-8aa3-1841a4541b55/bfe21baf-1342-48ad-994b-20326b13bad2"
-          (reference "#PWR024") (unit 1)
+          (reference "#PWR09") (unit 1)
         )
       )
@@
         )
         (path "/e63e39d7-6ac0-4ffd-8aa3-1841a4541b55/bfe21baf-1342-48ad-994b-20326b13bad2"
-          (reference "#PWR020") (unit 1)
+          (reference "#PWR05") (unit 1)
         )
       )
@@
       (effects (font (size 1.27 1.27)))
     )
-    (property "Footprint" "" (at 107.95 99.06 0)
+    (property "Footprint" "Package_DIP:DIP-24_W15.24mm_Socket" (at 107.95 99.06 0)
       (effects (font (size 1.27 1.27)) hide)
     )
@@
         )
         (path "/e63e39d7-6ac0-4ffd-8aa3-1841a4541b55/bfe21baf-1342-48ad-994b-20326b13bad2"
-          (reference "U8") (unit 1)
+          (reference "U3") (unit 1)
         )
       )
@@
         )
         (path "/e63e39d7-6ac0-4ffd-8aa3-1841a4541b55/bfe21baf-1342-48ad-994b-20326b13bad2"
-          (reference "U7") (unit 1)
+          (reference "U2") (unit 1)
         )
       )
@@
         )
         (path "/e63e39d7-6ac0-4ffd-8aa3-1841a4541b55/bfe21baf-1342-48ad-994b-20326b13bad2"
-          (reference "#PWR019") (unit 1)
+          (reference "#PWR04") (unit 1)
         )
       )
@@
       (effects (font (size 1.27 1.27)))
     )
-    (property "Footprint" "" (at 107.95 53.34 0)
+    (property "Footprint" "Package_DIP:DIP-24_W15.24mm_Socket" (at 107.95 53.34 0)
       (effects (font (size 1.27 1.27)) hide)
     )
@@
         )
         (path "/e63e39d7-6ac0-4ffd-8aa3-1841a4541b55/bfe21baf-1342-48ad-994b-20326b13bad2"
-          (reference "U6") (unit 1)
-        )
-      )
+          (reference "U1") (unit 1)
+        )
+      )
